File: kicad/MC34063InvertingEvalBoard.sch (KiCad schematic (older format))
At the start: 38 parts, among them P1 CONN_2, P2 CONN_2, U1 MC34063

Commit message: fixing a layout bug
Connections:
- net GND: no longer C5.2, U1.4 (GND)
- net at C6.2, C7.2, D1.1 (A)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: now also C5.2, U1.4 (GND)
Changed lines of the file:
@@
-	1    0    0    -1
-$EndComp
-$Comp
-L GND #PWR01
-U 1 1 554E7B3C
-P 9300 5550
-F 0 "#PWR01" H 9300 5550 30  0001 C CNN
-F 1 "GND" H 9300 5480 30  0001 C CNN
-F 2 "" H 9300 5550 60  0000 C CNN
-F 3 "" H 9300 5550 60  0000 C CNN
-	1    9300 5550
-	1    0    0    -1
-$EndComp
-$Comp
-L GND #PWR02
-U 1 1 554E7B55
-P 9000 5850
-F 0 "#PWR02" H 9000 5850 30  0001 C CNN
-F 1 "GND" H 9000 5780 30  0001 C CNN
-F 2 "" H 9000 5850 60  0000 C CNN
-F 3 "" H 9000 5850 60  0000 C CNN
-	1    9000 5850
 	1    0    0    -1
 $EndComp
@@
 	9400 5450 9300 5450
 Wire Wire Line
-	9300 5450 9300 5550
+	9300 5450 9300 5850
 Wire Wire Line
 	9000 5350 9000 5250
@@
 $EndComp
 $Comp
-L GND #PWR03
+L GND #PWR01
 U 1 1 554E7D7A
 P 1250 4450
-F 0 "#PWR03" H 1250 4450 30  0001 C CNN
+F 0 "#PWR01" H 1250 4450 30  0001 C CNN
 F 1 "GND" H 1250 4380 30  0001 C CNN
 F 2 "" H 1250 4450 60  0000 C CNN
@@
 	6150 4150 6150 4250
 $Comp
-L GND #PWR04
+L GND #PWR02
 U 1 1 554E7DA7
 P 6150 4750
-F 0 "#PWR04" H 6150 4750 30  0001 C CNN
+F 0 "#PWR02" H 6150 4750 30  0001 C CNN
 F 1 "GND" H 6150 4680 30  0001 C CNN
 F 2 "" H 6150 4750 60  0000 C CNN
@@
 $EndComp
 $Comp
-L GND #PWR05
+L GND #PWR03
 U 1 1 554E819B
 P 15550 7000
-F 0 "#PWR05" H 15550 7000 30  0001 C CNN
+F 0 "#PWR03" H 15550 7000 30  0001 C CNN
 F 1 "GND" H 15550 6930 30  0001 C CNN
 F 2 "" H 15550 7000 60  0000 C CNN
@@
 	14050 6700 15650 6700
 $Comp
-L GND #PWR06
+L GND #PWR04
 U 1 1 554E8260
 P 10200 6100
-F 0 "#PWR06" H 10200 6100 30  0001 C CNN
+F 0 "#PWR04" H 10200 6100 30  0001 C CNN
 F 1 "GND" H 10200 6030 30  0001 C CNN
 F 2 "" H 10200 6100 60  0000 C CNN
@@
 $EndComp
 $Comp
-L GND #PWR07
+L GND #PWR05
 U 1 1 554E8348
 P 11300 4750
-F 0 "#PWR07" H 11300 4750 30  0001 C CNN
+F 0 "#PWR05" H 11300 4750 30  0001 C CNN
 F 1 "GND" H 11300 4680 30  0001 C CNN
 F 2 "" H 11300 4750 60  0000 C CNN
@@
 Connection ~ 9600 6700
 $Comp
-L GND #PWR08
+L GND #PWR06
 U 1 1 554EE4DB
 P 9600 9600
-F 0 "#PWR08" H 9600 9600 30  0001 C CNN
+F 0 "#PWR06" H 9600 9600 30  0001 C CNN
 F 1 "GND" H 9600 9530 30  0001 C CNN
 F 2 "" H 9600 9600 60  0000 C CNN
@@
 $EndComp
 $Comp
-L GND #PWR09
+L GND #PWR07
 U 1 1 554EE7D5
 P 6500 4750
-F 0 "#PWR09" H 6500 4750 30  0001 C CNN
+F 0 "#PWR07" H 6500 4750 30  0001 C CNN
 F 1 "GND" H 6500 4680 30  0001 C CNN
 F 2 "" H 6500 4750 60  0000 C CNN
@@
 $EndComp
 $Comp
-L GND #PWR010
+L GND #PWR08
 U 1 1 554EE870
 P 10500 6100
-F 0 "#PWR010" H 10500 6100 30  0001 C CNN
+F 0 "#PWR08" H 10500 6100 30  0001 C CNN
 F 1 "GND" H 10500 6030 30  0001 C CNN
 F 2 "" H 10500 6100 60  0000 C CNN
@@
 $EndComp
 $Comp
-L GND #PWR011
+L GND #PWR09
 U 1 1 554EE90E
 P 14150 6100
-F 0 "#PWR011" H 14150 6100 30  0001 C CNN
+F 0 "#PWR09" H 14150 6100 30  0001 C CNN
 F 1 "GND" H 14150 6030 30  0001 C CNN
 F 2 "" H 14150 6100 60  0000 C CNN
@@
 $EndComp
 $Comp
-L GND #PWR012
+L GND #PWR010
 U 1 1 554EE91B
 P 14450 6100
-F 0 "#PWR012" H 14450 6100 30  0001 C CNN
+F 0 "#PWR010" H 14450 6100 30  0001 C CNN
 F 1 "GND" H 14450 6030 30  0001 C CNN
 F 2 "" H 14450 6100 60  0000 C CNN
@@
 $EndComp
 $Comp
-L GND #PWR013
+L GND #PWR011
 U 1 1 554EEAA0
 P 4200 4750
-F 0 "#PWR013" H 4200 4750 30  0001 C CNN
+F 0 "#PWR011" H 4200 4750 30  0001 C CNN
 F 1 "GND" H 4200 4680 30  0001 C CNN
 F 2 "" H 4200 4750 60  0000 C CNN
@@
 $EndComp
 $Comp
-L GND #PWR014
+L GND #PWR012
 U 1 1 554EEAAD
 P 4550 4750
-F 0 "#PWR014" H 4550 4750 30  0001 C CNN
+F 0 "#PWR012" H 4550 4750 30  0001 C CNN
 F 1 "GND" H 4550 4680 30  0001 C CNN
 F 2 "" H 4550 4750 60  0000 C CNN
@@
 	13350 6700 13450 6700
 $Comp
-L GND #PWR015
+L GND #PWR013
 U 1 1 554EF104
 P 15250 6300
-F 0 "#PWR015" H 15250 6300 30  0001 C CNN
+F 0 "#PWR013" H 15250 6300 30  0001 C CNN
 F 1 "GND" H 15250 6230 30  0001 C CNN
 F 2 "" H 15250 6300 60  0000 C CNN
@@
 $EndComp
 $Comp
-L GND #PWR016
+L GND #PWR014
 U 1 1 554EF220
 P 12350 6300
-F 0 "#PWR016" H 12350 6300 30  0001 C CNN
+F 0 "#PWR014" H 12350 6300 30  0001 C CNN
 F 1 "GND" H 12350 6230 30  0001 C CNN
 F 2 "" H 12350 6300 60  0000 C CNN
@@
 $EndComp
 $Comp
-L GND #PWR017
+L GND #PWR015
 U 1 1 554EF22E
 P 7450 3750
-F 0 "#PWR017" H 7450 3750 30  0001 C CNN
+F 0 "#PWR015" H 7450 3750 30  0001 C CNN
 F 1 "GND" H 7450 3680 30  0001 C CNN
 F 2 "" H 7450 3750 60  0000 C CNN
@@
 $EndComp
 $Comp
-L GND #PWR018
+L GND #PWR016
 U 1 1 554EF23C
 P 3750 3750
-F 0 "#PWR018" H 3750 3750 30  0001 C CNN
+F 0 "#PWR016" H 3750 3750 30  0001 C CNN
 F 1 "GND" H 3750 3680 30  0001 C CNN
 F 2 "" H 3750 3750 60  0000 C CNN
@@
 Connection ~ 10200 9500
 Connection ~ 9900 9500
+Wire Wire Line
+	9000 5850 10900 5850
+Wire Wire Line
+	10900 5850 10900 6700
+Connection ~ 10900 6700
+Connection ~ 9300 5850
 $EndSCHEMATC
